File: hardware/usbuc.sch (EAGLE design)
At the start: 14 parts, among them J1 PROGRAM, J2 DEVICE, U1 NCP551, U2 AT25SF081-XMHD-T, U3 PIC32MX250F128B-I_ML, Y1 8MHz

Commit message: Clear up crystal values in schematic
Parts:
- C1, C2: value 10pF -> 18pF; device SparkFun-Capacitors:10PF-0603-50V-5% -> SparkFun-Capacitors:18PF-0603-50V-5%
Other:
- note added: "ABM3B- 8.000MHZ- 10-1-U-T"
Changed lines of the file:
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@@
 <?xml version="1.0" encoding="utf-8"?>
 <!DOCTYPE eagle SYSTEM "eagle.dtd">
-<eagle version="6.5.0">
+<eagle version="8.6.2">
 <drawing>
 <settings>
 <setting alwaysvectorfont="no"/>
+<setting keepoldvectorfont="yes"/>
 <setting verticaltext="up"/>
 </settings>
@@
 <parts>
 <part name="Y1" library="SparkFun-Clocks" deviceset="CRYSTAL-8MHZ" device="SMD-5X3.2" value="8MHz"/>
-<part name="C1" library="SparkFun-Capacitors" deviceset="10PF" device="-0603-50V-5%" value="10pF"/>
-<part name="C2" library="SparkFun-Capacitors" deviceset="10PF" device="-0603-50V-5%" value="10pF"/>
 <part name="GND1" library="SparkFun-PowerSymbols" deviceset="GND" device=""/>
 <part name="SUPPLY2" library="SparkFun-PowerSymbols" deviceset="3.3V" device=""/>
@@
 <part name="SUPPLY6" library="SparkFun-PowerSymbols" deviceset="VIN" device=""/>
 <part name="FRAME1" library="SparkFun-Aesthetics" deviceset="FRAME-A4L" device=""/>
+<part name="C1" library="SparkFun-Capacitors" deviceset="18PF" device="-0603-50V-5%" value="18pF"/>
+<part name="C2" library="SparkFun-Capacitors" deviceset="18PF" device="-0603-50V-5%" value="18pF"/>
 </parts>
 <sheets>
@@
 <text x="194.564" y="1.27" size="2.54" layer="94" font="vector">1/1</text>
 <text x="235.204" y="1.27" size="2.54" layer="94" font="vector">1.0</text>
+<text x="38.354" y="70.104" size="1.27" layer="96" align="top-left">ABM3B-
+8.000MHZ-
+10-1-U-T</text>
 </plain>
 <instances>
@@
 <attribute name="NAME" x="41.656" y="79.502" size="1.778" layer="95" font="vector" rot="R180" align="bottom-center"/>
 <attribute name="VALUE" x="42.164" y="71.882" size="1.778" layer="96" font="vector" rot="R180" align="top-center"/>
-</instance>
-<instance part="C1" gate="G$1" x="33.02" y="81.28" smashed="yes" rot="R90">
-<attribute name="NAME" x="33.528" y="85.471" size="1.778" layer="95" font="vector" rot="R180"/>
-<attribute name="VALUE" x="35.56" y="78.867" size="1.778" layer="96" font="vector" rot="R180"/>
-</instance>
-<instance part="C2" gate="G$1" x="33.02" y="71.12" smashed="yes" rot="R90">
-<attribute name="NAME" x="33.528" y="75.565" size="1.778" layer="95" font="vector" rot="R180"/>
-<attribute name="VALUE" x="35.306" y="68.199" size="1.778" layer="96" font="vector" rot="R180"/>
 </instance>
 <instance part="GND1" gate="1" x="25.4" y="66.04"/>
@@
 <instance part="SUPPLY6" gate="G$1" x="233.68" y="73.66"/>
 <instance part="FRAME1" gate="G$1" x="0" y="0" smashed="yes"/>
+<instance part="C1" gate="G$1" x="33.02" y="81.28" smashed="yes" rot="R90">
+<attribute name="NAME" x="33.528" y="85.471" size="1.778" layer="95" font="vector" rot="R180"/>
+<attribute name="VALUE" x="35.814" y="78.867" size="1.778" layer="96" font="vector" rot="R180"/>
+</instance>
+<instance part="C2" gate="G$1" x="33.02" y="71.12" smashed="yes" rot="R90">
+<attribute name="NAME" x="33.528" y="75.311" size="1.778" layer="95" font="vector" rot="R180"/>
+<attribute name="VALUE" x="35.56" y="68.453" size="1.778" layer="96" font="vector" rot="R180"/>
+</instance>
 </instances>
 <busses>
@@
 <wire x1="45.72" y1="81.28" x2="38.1" y2="81.28" width="0.1524" layer="91"/>
 <wire x1="38.1" y1="81.28" x2="38.1" y2="78.74" width="0.1524" layer="91"/>
-<wire x1="38.1" y1="81.28" x2="35.56" y2="81.28" width="0.1524" layer="91"/>
-<pinref part="C1" gate="G$1" pin="2"/>
 <pinref part="U3" gate="A" pin="OSC1/CLKI/RPA2/RA2"/>
 <wire x1="58.42" y1="78.74" x2="45.72" y2="78.74" width="0.1524" layer="91"/>
 <junction x="38.1" y="81.28"/>
+<pinref part="C1" gate="G$1" pin="2"/>
+<wire x1="38.1" y1="81.28" x2="35.56" y2="81.28" width="0.1524" layer="91"/>
 </segment>
 </net>
@@
 <wire x1="45.72" y1="71.12" x2="38.1" y2="71.12" width="0.1524" layer="91"/>
 <wire x1="38.1" y1="71.12" x2="38.1" y2="73.66" width="0.1524" layer="91"/>
-<wire x1="38.1" y1="71.12" x2="35.56" y2="71.12" width="0.1524" layer="91"/>
-<pinref part="C2" gate="G$1" pin="2"/>
 <pinref part="U3" gate="A" pin="OSC2/CLKO/RPA3/PMA0/RA3"/>
 <wire x1="45.72" y1="76.2" x2="58.42" y2="76.2" width="0.1524" layer="91"/>
 <junction x="38.1" y="71.12"/>
+<pinref part="C2" gate="G$1" pin="2"/>
+<wire x1="38.1" y1="71.12" x2="35.56" y2="71.12" width="0.1524" layer="91"/>
 </segment>
 </net>
 <net name="GND" class="0">
 <segment>
-<pinref part="C1" gate="G$1" pin="1"/>
-<wire x1="27.94" y1="81.28" x2="25.4" y2="81.28" width="0.1524" layer="91"/>
 <wire x1="25.4" y1="81.28" x2="25.4" y2="71.12" width="0.1524" layer="91"/>
-<pinref part="C2" gate="G$1" pin="1"/>
-<wire x1="27.94" y1="71.12" x2="25.4" y2="71.12" width="0.1524" layer="91"/>
 <wire x1="25.4" y1="71.12" x2="25.4" y2="68.58" width="0.1524" layer="91"/>
 <pinref part="GND1" gate="1" pin="GND"/>
@@
 <junction x="25.4" y="71.12"/>
 <label x="2.54" y="93.98" size="1.778" layer="95"/>
+<pinref part="C1" gate="G$1" pin="1"/>
+<wire x1="27.94" y1="81.28" x2="25.4" y2="81.28" width="0.1524" layer="91"/>
+<pinref part="C2" gate="G$1" pin="1"/>
+<wire x1="27.94" y1="71.12" x2="25.4" y2="71.12" width="0.1524" layer="91"/>
 </segment>
 <segment>
@@
 </schematic>
 </drawing>
+<compatibility>
+<note version="6.3" minversion="6.2.2" severity="warning">
+Since Version 6.2.2 text objects can contain more than one line,
+which will not be processed correctly with this version.
+</note>
+</compatibility>
 </eagle>
